Commit message: Finished part 3

File: xacro/barista_robot_model.urdf.xacro (robot description, xacro)
@@ -12,4 +12,6 @@
 <xacro:arg name="include_laser" default="true"/>
 <xacro:property name="include_laser" value="$(arg include_laser)" />
+<xacro:arg name="robot_name" default="barista"/>
+<xacro:property name="robot_name" value="$(arg robot_name)" />
 <!-- Colors -->
 <material name="red">
@@ -296,4 +298,5 @@
         <plugin name="barista_joint_state" filename="libgazebo_ros_joint_state_publisher.so">
             <ros>
+                <namespace>/${robot_name}</namespace>
                 <remapping>~/out:=joint_states</remapping>
             </ros>
@@ -324,40 +327,15 @@
             <publish_odom>true</publish_odom>
             <publish_odom_tf>true</publish_odom_tf>
-            <odometry_frame>odom</odometry_frame>
-            <robot_base_frame>base_link</robot_base_frame>
+            <publish_wheel_tf>false</publish_wheel_tf>
+            <ros>
+                <namespace>/${robot_name}</namespace>
+                <remapping>/cmd_vel:=cmd_vel</remapping>
+            </ros>
+            <odometry_frame>${robot_name}/odom</odometry_frame>
+            <robot_base_frame>${robot_name}/base_link</robot_base_frame>
         </plugin>
     </gazebo>
     <xacro:if value="${include_laser}">
-        <!-- Laser scan link -->
-        <link name="laser_scan_link">
-            <visual>
-                <origin xyz="0 0 0" rpy="0 0 0"/>
-                <geometry>
-                    <!--<mesh filename="../meshes/rplidar.dae"/>-->
-                    <mesh filename="package://barista_robot_description/meshes/rplidar.dae" scale="1.0 1.0 1.0"/>
-                </geometry>
-            </visual>
-            <collision>
-                <origin xyz="0 0 0" rpy="0 0 0"/>
-                <geometry>
-                    <!--<mesh filename="../meshes/rplidar.dae"/>-->
-                    <mesh filename="package://barista_robot_description/meshes/rplidar.dae" scale="1.0 1.0 1.0"/>
-                </geometry>
-            </collision>
-            <inertial>
-                <mass value="0.3"/>
-                <origin xyz="0 0 0" rpy="0 0 0"/>
-                <inertia ixx="0.000001" ixy="0" ixz="0" iyy="0.000001" iyz="0" izz="0.000001"/>
-            </inertial>
-        </link>
-        <gazebo reference="laser_scan_link">
-            <material>Gazebo/Black</material>
-        </gazebo>
-        <joint name = "laser_scan_link_joint" type ="fixed">
-            <origin xyz="0 0 0.075" rpy="0 0 0"/>
-            <parent link = "chassis" />
-            <child link = "laser_scan_link" />
-        </joint>
-        <xacro:laser_scan_plugin link_name = "laser_scan_link"/>
+        <xacro:laser_scan_plugin  robot_name="${robot_name}"/>
     </xacro:if>
 </robot>

File: xacro/laser_scan.xacro (robot description, xacro)
@@ -1,7 +1,34 @@
 <?xml version="1.0"?>
 <robot xmlns:xacro="http://www.ros.org/wiki/xacro">
-<xacro:macro name="laser_scan_plugin" params="link_name">
+<xacro:macro name="laser_scan_plugin" params="robot_name">
+    <!-- Laser scan link -->
+    <link name="laser_scan_link">
+        <visual>
+            <origin xyz="0 0 0" rpy="0 0 0"/>
+            <geometry>
+                <!--<mesh filename="../meshes/rplidar.dae"/>-->
+                <mesh filename="package://barista_robot_description/meshes/rplidar.dae" scale="1.0 1.0 1.0"/>
+            </geometry>
+        </visual>
+        <collision>
+            <origin xyz="0 0 0" rpy="0 0 0"/>
+            <geometry>
+                <!--<mesh filename="../meshes/rplidar.dae"/>-->
+                <mesh filename="package://barista_robot_description/meshes/rplidar.dae" scale="1.0 1.0 1.0"/>
+            </geometry>
+        </collision>
+        <inertial>
+            <mass value="0.3"/>
+            <origin xyz="0 0 0" rpy="0 0 0"/>
+            <inertia ixx="0.000001" ixy="0" ixz="0" iyy="0.000001" iyz="0" izz="0.000001"/>
+        </inertial>
+    </link>
+    <joint name = "laser_scan_link_joint" type ="fixed">
+        <origin xyz="0 0 0.075" rpy="0 0 0"/>
+        <parent link = "chassis" />
+        <child link = "laser_scan_link" />
+    </joint>
     <!-- Laser scan plugin -->
-    <gazebo reference="${link_name}">
+    <gazebo reference="laser_scan_link">
         <sensor name="sensor_ray" type="ray">
             <pose>0 0 0 0 0 0</pose>
@@ -22,12 +49,15 @@
             <always_on>true</always_on>
             <visualize>false</visualize>
-            <update_rate>10.0</update_rate>
+            <update_rate>20.0</update_rate>
             <plugin name="laser" filename="libgazebo_ros_ray_sensor.so">
             <ros>
-                <remapping>~/out:=/scan</remapping>
+                <namespace>/${robot_name}</namespace>
+                <remapping>~/out:=scan</remapping>
             </ros>
             <output_type>sensor_msgs/LaserScan</output_type>
+            <frame_name>${robot_name}/laser_scan_link</frame_name>
             </plugin>
         </sensor>
+        <material>Gazebo/Black</material>
     </gazebo>
 </xacro:macro>
